File: project/_autosave-project.kicad_pcb (KiCad board)
At the start: 2 copper layers, 43.2 x 27.9 mm, 20 parts, among them P1 CONN_01X10, P2 CONN_02X06, P3 CONN_01X10, U1 iCE40-HX1K-VQ100, U2 TPS62207DBV, U3 Si501-PKG-B

Commit message: Version 0.3
Parts:
- removed L1: 10 uH, Capacitors_SMD:C_0805_HandSoldering
- added W4: TEST_1V2, Connect:PINTST, F.Cu at (168.1, 105.7)
- C4: value 4.7uF -> 100nF
- U2: value TPS62207DBV -> LD1117S12CTR; footprint TO_SOT_Packages_SMD:SOT-23-5 -> SOT-223
- moved W1 7.82 mm to (146.6, 97.0)
- moved D1 4.19 mm to (156.5, 120.1)
- moved R2 4.19 mm to (161.5, 120.1)
- moved W2 3.66 mm to (138.9, 119.9)
- moved W3 2.27 mm to (141.0, 119.9)
- moved U2 2.18 mm to (143.0, 104.9)
- moved C3 1.17 mm to (168.1, 109.5)
- moved R1 0.18 mm to (150.4, 120.1)
- moved D2 0.18 mm to (145.3, 120.1)
Connections:
- P1 pad 3: Net-(P1-Pad3) -> (no net)
- P1 pad 4: Net-(P1-Pad4) -> (no net)
- U1 pad 100: Net-(U1-Pad100) -> (no net)
- U1 pad 24: LED1 -> (no net)
- U1 pad 25: LED2 -> (no net)
- U1 pad 26: Net-(U1-Pad26) -> (no net)
- U1 pad 27: Net-(U1-Pad27) -> (no net)
- U1 pad 28: Net-(U1-Pad28) -> (no net)
- U1 pad 29: Net-(U1-Pad29) -> (no net)
- U1 pad 30: Net-(U1-Pad30) -> (no net)
- U1 pad 33: Net-(U1-Pad33) -> (no net)
- U1 pad 34: Net-(U1-Pad34) -> (no net)
- U1 pad 36: Net-(U1-Pad36) -> (no net)
- U1 pad 37: Net-(U1-Pad37) -> (no net)
- U1 pad 40: Net-(U1-Pad40) -> (no net)
- U1 pad 41: Net-(U1-Pad41) -> (no net)
- U1 pad 42: Net-(U1-Pad42) -> (no net)
- U1 pad 51: Net-(U1-Pad51) -> (no net)
- U1 pad 52: Net-(U1-Pad52) -> (no net)
- U1 pad 53: Net-(U1-Pad53) -> (no net)
- U1 pad 54: Net-(U1-Pad54) -> (no net)
- U1 pad 56: Net-(U1-Pad56) -> (no net)
- U1 pad 57: Net-(U1-Pad57) -> (no net)
- U1 pad 59: Net-(U1-Pad59) -> LED1
- U1 pad 60: Net-(U1-Pad60) -> (no net)
- U1 pad 62: Net-(U1-Pad62) -> (no net)
- U1 pad 63: Net-(U1-Pad63) -> (no net)
- U1 pad 64: Net-(U1-Pad64) -> (no net)
- U1 pad 65: Net-(U1-Pad65) -> (no net)
- U1 pad 66: Net-(U1-Pad66) -> (no net)
- U1 pad 68: Net-(U1-Pad68) -> (no net)
- U1 pad 69: Net-(U1-Pad69) -> (no net)
- U1 pad 71: Net-(U1-Pad71) -> (no net)
- U1 pad 72: Net-(U1-Pad72) -> (no net)
- U1 pad 73: Net-(U1-Pad73) -> (no net)
- U1 pad 74: Net-(U1-Pad74) -> LED2
- U1 pad 76: Net-(U1-Pad76) -> (no net)
- U1 pad 78: Net-(U1-Pad78) -> (no net)
- U1 pad 79: Net-(U1-Pad79) -> (no net)
- U1 pad 80: Net-(U1-Pad80) -> (no net)
- U1 pad 81: Net-(U1-Pad81) -> (no net)
- U1 pad 82: Net-(U1-Pad82) -> (no net)
- U1 pad 83: Net-(U1-Pad83) -> (no net)
- U1 pad 85: Net-(U1-Pad85) -> (no net)
- U1 pad 86: Net-(U1-Pad86) -> (no net)
- U1 pad 87: Net-(U1-Pad87) -> (no net)
- U1 pad 89: Net-(U1-Pad89) -> (no net)
- U1 pad 91: Net-(U1-Pad91) -> (no net)
- U1 pad 93: Net-(U1-Pad93) -> (no net)
- U1 pad 94: Net-(U1-Pad94) -> (no net)
- U1 pad 95: Net-(U1-Pad95) -> (no net)
- U1 pad 96: Net-(U1-Pad96) -> (no net)
- U1 pad 97: Net-(U1-Pad97) -> (no net)
- U1 pad 99: Net-(U1-Pad99) -> (no net)
- U2 pad 1: BANK_IO -> GND
- U2 pad 2: GND -> +1V2
- U2 pad 4: +1V2 -> (no net)
Routing:
- net LED2: track 29.3 -> 10.6 mm, vias 4 -> 2
- net +1V2: track 67.6 -> 51.3 mm
- net LED1: track 23.1 -> 8.46 mm, vias 4 -> 2
- net GND: track 194.1 -> 204.0 mm, vias 17 -> 16
- net Net-(L1-Pad1): track 3.63 -> 0.00 mm
- net BANK_IO: track 178.4 -> 175.6 mm
- net Net-(U1-Pad90): track 9.52 -> 11.8 mm
- net CDONE: track 23.5 -> 24.0 mm
Other:
- board text added: "tessel-fpga 0.3"
- board text removed: "tessel-fpga 0.2"
